Commit message: remove comment plate

File: robots/youbot_dual_arm.urdf.xacro (robot description, xacro)
@@ -32,7 +32,4 @@
   <!-- foot for arm-->
   <xacro:youbot_base name="base"/>
-  <!--<xacro:youbot_plate name="plate" parent="base_link">
-    <origin xyz="-0.159 0 0.046" rpy="0 0 0" />
-  </xacro:youbot_plate>-->
   <xacro:youbot_arm name="arm" parent="base_link">
     <!--<origin xyz="0.143 0 0.046" rpy="0 0 0" />-->
