Commit message: change to planar move controller + format

File: urdf/youbot_base/base.gazebo.xacro (robot description, xacro)
@@ -4,50 +4,46 @@
        xmlns:interface="http://playerstage.sourceforge.net/gazebo/xmlschema/#interface"
        xmlns:xacro="http://ros.org/wiki/xacro">
-	<xacro:macro name="youbot_base_gazebo">
-		<gazebo reference="youbot_base">
-     			<material value="youbot/DarkGrey" />
-    		</gazebo>
-	<!-- front left wheel -->
-    		<gazebo reference="wheel_link_fl">
-       			<material value="youbot/Orange" />
-    		</gazebo>
-    		<gazebo reference="caster_link_fl">
-      			<material value="youbot/Orange" />
-    		</gazebo>
-	<!-- front right wheel -->
-    		<gazebo reference="wheel_link_fr">
-       			<material value="youbot/Orange" />
-    		</gazebo>
-    		<gazebo reference="caster_link_fr">
-      			<material value="youbot/Orange" />
-    		</gazebo>
-	<!-- back left wheel -->
-    		<gazebo reference="wheel_link_bl">
-       			<material value="youbot/Orange" />
-    		</gazebo>
-    		<gazebo reference="caster_link_bl">
-      			<material value="youbot/Orange" />
-    		</gazebo>
-	<!-- back right wheel -->
-    		<gazebo reference="wheel_link_br">
-       			<material value="youbot/Orange" />
-    		</gazebo>
-    		<gazebo reference="caster_link_br">
-      			<material value="youbot/Orange" />
-    		</gazebo>
-	<!-- position controller -->
-		<gazebo>
-      			<plugin name="p3d_base_controller" filename="libgazebo_ros_p3d.so">
-        			<alwaysOn>true</alwaysOn>
-        			<updateRate>100.0</updateRate>
-        			<bodyName>base_link</bodyName>
-        			<topicName>base_pose_ground_truth</topicName>
-        			<gaussianNoise>0.01</gaussianNoise>
-        			<frameName>map</frameName>
-        			<xyzOffsets>25.7 25.7 0</xyzOffsets> <!-- initialize odometry for fake localization-->
-        			<rpyOffsets>0 0 0</rpyOffsets>
-      			</plugin>
-      			<canonicalBody>base_footprint</canonicalBody>
-    		</gazebo>
+  <xacro:macro name="youbot_base_gazebo">
+    <gazebo reference="youbot_base">
+      <material value="youbot/DarkGrey" />
+    </gazebo>
+    <!-- front left wheel -->
+    <gazebo reference="wheel_link_fl">
+      <material value="youbot/Orange" />
+    </gazebo>
+    <gazebo reference="caster_link_fl">
+      <material value="youbot/Orange" />
+    </gazebo>
+    <!-- front right wheel -->
+    <gazebo reference="wheel_link_fr">
+      <material value="youbot/Orange" />
+    </gazebo>
+    <gazebo reference="caster_link_fr">
+      <material value="youbot/Orange" />
+    </gazebo>
+    <!-- back left wheel -->
+    <gazebo reference="wheel_link_bl">
+      <material value="youbot/Orange" />
+    </gazebo>
+    <gazebo reference="caster_link_bl">
+      <material value="youbot/Orange" />
+    </gazebo>
+    <!-- back right wheel -->
+    <gazebo reference="wheel_link_br">
+      <material value="youbot/Orange" />
+    </gazebo>
+    <gazebo reference="caster_link_br">
+      <material value="youbot/Orange" />
+    </gazebo>
+    <!-- position controller -->
+    <gazebo>
+      <plugin name="base_controller" filename="libgazebo_ros_planar_move.so">
+        <commandTopic>cmd_vel</commandTopic>
+        <odometryTopic>odom</odometryTopic>
+        <odometryFrame>odom</odometryFrame>
+        <odometryRate>100.0</odometryRate>
+        <robotBaseFrame>base_link</robotBaseFrame>
+      </plugin>
+    </gazebo>
   </xacro:macro>
 </robot>
