Commit message: update  interias of the arm

File: urdf/youbot_arm/limits.urdf.xacro (robot description, xacro)
@@ -35,30 +35,30 @@
 		<origin xyz="0 0 0"
 			rpy="0 0 0" />
-		<inertia ixx="0.1" ixy="0" ixz="0" iyy="0.1" iyz="0" izz="0.1" />
+		<inertia ixx="1.0" ixy="0.0" ixz="0.0" iyy="1.0" iyz="0.0" izz="1.0"/>
 	</xacro:macro>
 	<xacro:macro name="link_1_inertia_tensor">
 		<origin xyz="${14.89/1000} ${2.13/1000} ${2.13/1000}"
 			rpy="0 0 0" />
-		<inertia ixx="0.003863" ixy="-0.000979" ixz="0.000000" iyy="0.006196" iyz="0.000000" izz="0.006369" />
+		<inertia ixx="0.0029525" ixy="0.0" ixz="0.0" iyy="0.0060091" iyz="0.0" izz="0.0058821"/>
 	</xacro:macro>
 	<xacro:macro name="link_2_inertia_tensor">
-		<origin xyz="${104.53/1000} ${1.7/1000} ${-2.97/1000}"
+		<origin xyz="${10.53/1000} ${-30.7/1000} ${85.97/1000}"
 			rpy="0 0 0" />
-		<inertia ixx="0.000823" ixy="0.000000" ixz="-0.000000" iyy="0.004447" iyz ="0.000000" izz="0.004439" />
+		<inertia ixx="0.0031145" ixy="0.0" ixz="0.0" iyy="0.0005843" iyz="0.0" izz="0.0031631"/>
 	</xacro:macro>
 	<xacro:macro name="link_3_inertia_tensor">
-		<origin xyz="${0.1/1000} ${96.7/1000} ${21.07/1000}"
+		<origin xyz="${0.1/1000} ${20.7/1000} ${71.07/1000}"
 			rpy="0 0 0" />
-		<inertia ixx="0.002459" ixy="0.000000" ixz="0.000000" iyy="0.002571" iyz="-0.000000" izz="0.000535" />
+		<inertia ixx="0.00172767" ixy="0.0" ixz="0.0" iyy="0.00041967" iyz="0.0" izz="0.0018468"/>
 	</xacro:macro>
 	<xacro:macro name="link_4_inertia_tensor">
-		<origin xyz="${0.11/1000} ${51.03/1000} ${-23.19/1000}"
+		<origin xyz="${0.11/1000} ${-20.0/1000} ${50.19/1000}"
 			rpy="0 0 0"  />
-		<inertia ixx="0.000869" ixy="0.000000" ixz="-0.000000" iyy="0.001173" iyz="-0.000231" izz="0.001091" />
+		<inertia ixx="0.0006764" ixy="0.0" ixz="0.0" iyy="0.0010573" iyz="0.0" izz="0.0006610"/>
 	</xacro:macro>
 	<xacro:macro name="link_5_inertia_tensor">
 		<origin xyz="${0/1000} ${1.15/1000} ${-16.83/1000}"
 			rpy="0 0 0" />
-		<inertia ixx="0.000280" ixy="0.000000" ixz="0.000000" iyy="0.000339" iyz="0.000000" izz="0.000119" />
+		<inertia ixx="0.0001934" ixy="0.0" ixz="0.0" iyy="0.0001602" iyz="0.0" izz="0.0000689"/>
 	</xacro:macro>
 </robot>

Commit message: correct formatting

File: urdf/youbot_arm/limits.urdf.xacro (robot description, xacro)
@@ -3,5 +3,5 @@
 	<!-- common properties -->
 	<property name="M_PI" value="3.1415926535897931" />
-        <property name="threshold" value="0.01" />
+	<property name="threshold" value="0.01" />
 	<!-- arm limits positions (deg) -->
 	<property name="joint_1_limit" value="${M_PI * (169 + 169) / 180}" />
@@ -10,5 +10,5 @@
 	<property name="joint_4_limit" value="${M_PI * (102.5 + 102.5) / 180}" />
 	<property name="joint_5_limit" value="${M_PI * (167.5 + 167.5) / 180}" />
-        <property name="joint_1_limit_soft" value="${M_PI * (169 + 169) / 180 - threshold}" />
+	<property name="joint_1_limit_soft" value="${M_PI * (169 + 169) / 180 - threshold}" />
 	<property name="joint_2_limit_soft" value="${M_PI * (90 + 65) / 180 - threshold}" />
 	<property name="joint_3_limit_soft" value="${M_PI * (146 + 151) / 180 - threshold}" />
@@ -30,5 +30,5 @@
 	<!-- TODO: add inertia tensor-->
 	<xacro:macro name="default_origin">
-        	<origin xyz="0 0 0" rpy="0 0 0"/> <!-- no data known -->
+		<origin xyz="0 0 0" rpy="0 0 0"/> <!-- no data known -->
 	</xacro:macro>
 	<xacro:macro name="link_default_inertia_tensor">
