Commit message: use new syntax to include a transmission

File: urdf/youbot_arm/arm.transmission.xacro (robot description, xacro)
@@ -7,28 +7,43 @@
 	<!-- reduction ratio must not to be 0-->
 	<xacro:macro name="youbot_arm_transmission" params="name">
-		<transmission name="${name}_trans_1" type="pr2_mechanism_model/SimpleTransmission">
-			<actuator name="${name}_motor_1"/>
+		<transmission name="${name}_trans_1">
+      <type>transmission_interface/SimpleTransmission</type>
+			<actuator name="${name}_motor_1">
+        <hardwareInterface>EffortJointInterface</hardwareInterface>
+        <mechanicalReduction>1</mechanicalReduction>
+      </actuator>
 			<joint name="${name}_joint_1"/>
-			<mechanicalReduction>1</mechanicalReduction>
 		</transmission>
-		<transmission name="${name}_trans_2" type="pr2_mechanism_model/SimpleTransmission">
-			<actuator name="${name}_motor_2"/>
+		<transmission name="${name}_trans_2">
+      <type>transmission_interface/SimpleTransmission</type>
+			<actuator name="${name}_motor_2">
+        <hardwareInterface>EffortJointInterface</hardwareInterface>
+        <mechanicalReduction>1</mechanicalReduction>
+      </actuator>
 			<joint name="${name}_joint_2"/>
-			<mechanicalReduction>1</mechanicalReduction>
 		</transmission>
-		<transmission name="${name}_trans_3" type="pr2_mechanism_model/SimpleTransmission">
-			<actuator name="${name}_motor_3"/>
+		<transmission name="${name}_trans_3">
+      <type>transmission_interface/SimpleTransmission</type>
+			<actuator name="${name}_motor_3">
+        <hardwareInterface>EffortJointInterface</hardwareInterface>
+        <mechanicalReduction>1</mechanicalReduction>
+      </actuator>
 			<joint name="${name}_joint_3"/>
-			<mechanicalReduction>1</mechanicalReduction>
 		</transmission>
-		<transmission name="${name}_trans_4" type="pr2_mechanism_model/SimpleTransmission">
-			<actuator name="${name}_motor_4"/>
+		<transmission name="${name}_trans_4">
+      <type>transmission_interface/SimpleTransmission</type>
+			<actuator name="${name}_motor_4">
+        <hardwareInterface>EffortJointInterface</hardwareInterface>
+        <mechanicalReduction>1</mechanicalReduction>
+      </actuator>
 			<joint name="${name}_joint_4"/>
-			<mechanicalReduction>1</mechanicalReduction>
 		</transmission>
-		<transmission name="${name}_trans_5" type="pr2_mechanism_model/SimpleTransmission">
-			<actuator name="${name}_motor_5"/>
+		<transmission name="${name}_trans_5">
+      <type>transmission_interface/SimpleTransmission</type>
+			<actuator name="${name}_motor_5">
+        <hardwareInterface>EffortJointInterface</hardwareInterface>
+        <mechanicalReduction>1</mechanicalReduction>
+      </actuator>
 			<joint name="${name}_joint_5"/>
-			<mechanicalReduction>1</mechanicalReduction>
 		</transmission>
 	</xacro:macro>

File: urdf/youbot_base/base.transmission.xacro (robot description, xacro)
@@ -6,50 +6,78 @@
 	<property name="wheel_mechanical_reduction" value="${624/35 * 80/18}" />
 	<property name="caster_mechanical_reduction" value="${624/35 * 80/18}" />
-  	<property name="" value="0.360" />
+  <property name="" value="0.360" />
 	<xacro:macro name="youbot_base_transmission">
 	<!-- front left wheel -->
-		<transmission name="wheel_trans_fl" type="pr2_mechanism_model/SimpleTransmission">
-			<actuator name="wheel_motor_fl" />
+		<transmission name="wheel_trans_fl">
+      <type>transmission_interface/SimpleTransmission</type>
+			<actuator name="wheel_motor_fl">
+        <hardwareInterface>VelocityJointInterface</hardwareInterface>
+        <mechanicalReduction>${wheel_mechanical_reduction}</mechanicalReduction>
+      </actuator>
 			<joint name="wheel_joint_fl" />
 			<mechanicalReduction>${wheel_mechanical_reduction}</mechanicalReduction>
 		</transmission>
-		<transmission name="caster_trans_fl" type="pr2_mechanism_model/SimpleTransmission">
-      			<actuator name="caster_motor_fl" />
-      			<joint name="caster_joint_fl" />
-      			<mechanicalReduction>${caster_mechanical_reduction}</mechanicalReduction>
-    		</transmission>
-	<!-- front right wheel -->
-		<transmission name="wheel_trans_fr" type="pr2_mechanism_model/SimpleTransmission">
-			<actuator name="wheel_motor_fr" />
-			<joint name="wheel_joint_fr" />
-			<mechanicalReduction>${wheel_mechanical_reduction}</mechanicalReduction>
-		</transmission>
-		<transmission name="caster_trans_fr" type="pr2_mechanism_model/SimpleTransmission">
-      			<actuator name="caster_motor_fr" />
-      			<joint name="caster_joint_fr" />
-      			<mechanicalReduction>${caster_mechanical_reduction}</mechanicalReduction>
-    		</transmission>
-	<!-- back left wheel -->
-		<transmission name="wheel_trans_bl" type="pr2_mechanism_model/SimpleTransmission">
-			<actuator name="wheel_motor_bl" />
-			<joint name="wheel_joint_bl" />
-			<mechanicalReduction>${wheel_mechanical_reduction}</mechanicalReduction>
-		</transmission>
-		<transmission name="caster_trans_bl" type="pr2_mechanism_model/SimpleTransmission">
-      			<actuator name="caster_motor_bl" />
-      			<joint name="caster_joint_bl" />
-      			<mechanicalReduction>${caster_mechanical_reduction}</mechanicalReduction>
-    		</transmission>
-	<!-- back right wheel -->
-		<transmission name="wheel_trans_br" type="pr2_mechanism_model/SimpleTransmission">
-			<actuator name="wheel_motor_br" />
-			<joint name="wheel_joint_br" />
-			<mechanicalReduction>${wheel_mechanical_reduction}</mechanicalReduction>
-		</transmission>
-		<transmission name="caster_trans_br" type="pr2_mechanism_model/SimpleTransmission">
-      			<actuator name="caster_motor_br" />
-      			<joint name="caster_joint_br" />
-      			<mechanicalReduction>${caster_mechanical_reduction}</mechanicalReduction>
-    		</transmission>
-  	</xacro:macro>
+		<transmission name="caster_trans_fl">
+      <type>transmission_interface/SimpleTransmission</type>
+   	  <actuator name="caster_motor_fl">
+        <hardwareInterface>VelocityJointInterface</hardwareInterface>
+        <mechanicalReduction>${wheel_mechanical_reduction}</mechanicalReduction>
+      </actuator>
+      <joint name="caster_joint_fl" />
+      <mechanicalReduction>${caster_mechanical_reduction}</mechanicalReduction>
+    </transmission>
+	  <!-- front right wheel -->
+	  <transmission name="wheel_trans_fr">
+      <type>transmission_interface/SimpleTransmission</type>
+		  <actuator name="wheel_motor_fr">
+        <hardwareInterface>VelocityJointInterface</hardwareInterface>
+        <mechanicalReduction>${wheel_mechanical_reduction}</mechanicalReduction>
+      </actuator>
+		  <joint name="wheel_joint_fr" />
+		  <mechanicalReduction>${wheel_mechanical_reduction}</mechanicalReduction>
+	  </transmission>
+	  <transmission name="caster_trans_fr">
+      <type>transmission_interface/SimpleTransmission</type>
+      <actuator name="caster_motor_fr" >
+        <hardwareInterface>VelocityJointInterface</hardwareInterface>
+        <mechanicalReduction>${wheel_mechanical_reduction}</mechanicalReduction>
+      </actuator>
+    	<joint name="caster_joint_fr" />
+    	<mechanicalReduction>${caster_mechanical_reduction}</mechanicalReduction>
+    </transmission>
+	  <!-- back left wheel -->
+	  <transmission name="wheel_trans_bl">
+      <type>transmission_interface/SimpleTransmission</type>
+	    <actuator name="wheel_motor_bl" >
+        <hardwareInterface>VelocityJointInterface</hardwareInterface>
+        <mechanicalReduction>${wheel_mechanical_reduction}</mechanicalReduction>
+      </actuator>
+	    <joint name="wheel_joint_bl" />
+	  </transmission>
+	  <transmission name="caster_trans_bl">
+      <type>transmission_interface/SimpleTransmission</type>
+      <actuator name="caster_motor_bl" >
+        <hardwareInterface>VelocityJointInterface</hardwareInterface>
+        <mechanicalReduction>${wheel_mechanical_reduction}</mechanicalReduction>
+      </actuator>
+    	<joint name="caster_joint_bl" />
+    </transmission>
+	  <!-- back right wheel -->
+	  <transmission name="wheel_trans_br">
+      <type>transmission_interface/SimpleTransmission</type>
+	    <actuator name="wheel_motor_br" >
+        <hardwareInterface>VelocityJointInterface</hardwareInterface>
+        <mechanicalReduction>${wheel_mechanical_reduction}</mechanicalReduction>
+      </actuator>
+		  <joint name="wheel_joint_br" />
+	  </transmission>
+	  <transmission name="caster_trans_br">
+      <type>transmission_interface/SimpleTransmission</type>
+      <actuator name="caster_motor_br" >
+        <hardwareInterface>VelocityJointInterface</hardwareInterface>
+        <mechanicalReduction>${wheel_mechanical_reduction}</mechanicalReduction>
+      </actuator>
+    	<joint name="caster_joint_br" />
+    </transmission>
+  </xacro:macro>
 </robot>

File: urdf/youbot_gripper/gripper.transmission.xacro (robot description, xacro)
@@ -5,13 +5,19 @@
        xmlns:xacro="http://ros.org/wiki/xacro">
 	<xacro:macro name="youbot_gripper_transmission" params="name">
-		<transmission name="${name}_finger_l_trans" type="pr2_mechanism_model/SimpleTransmission">
-			<actuator name="${name}_finger_l_motor"/>
+		<transmission name="${name}_finger_l_trans">
+      <type>transmission_interface/SimpleTransmission</type>
+			<actuator name="${name}_finger_l_motor">
+        <hardwareInterface>EffortJointInterface</hardwareInterface>
+        <mechanicalReduction>1</mechanicalReduction>
+      </actuator>
 			<joint name="${name}_finger_joint_l"/>
-			<mechanicalReduction>1</mechanicalReduction>
 		</transmission>
-		<transmission name="${name}_finger_r_trans" type="pr2_mechanism_model/SimpleTransmission">
-			<actuator name="${name}_finger_r_motor"/>
+		<transmission name="${name}_finger_r_trans">
+      <type>transmission_interface/SimpleTransmission</type>
+			<actuator name="${name}_finger_r_motor">
+        <hardwareInterface>EffortJointInterface</hardwareInterface>
+        <mechanicalReduction>1</mechanicalReduction>
+      </actuator>
 			<joint name="${name}_finger_joint_r"/>
-			<mechanicalReduction>1</mechanicalReduction>
 		</transmission>
 	</xacro:macro>

Commit message: fix indentation

File: urdf/youbot_arm/arm.transmission.xacro (robot description, xacro)
@@ -4,47 +4,47 @@
        xmlns:interface="http://playerstage.sourceforge.net/gazebo/xmlschema/#interface"
        xmlns:xacro="http://ros.org/wiki/xacro">
-	<!-- reduction ratio doesn't affect the model-->
-	<!-- reduction ratio must not to be 0-->
-	<xacro:macro name="youbot_arm_transmission" params="name">
-		<transmission name="${name}_trans_1">
+  <!-- reduction ratio doesn't affect the model-->
+  <!-- reduction ratio must not to be 0-->
+  <xacro:macro name="youbot_arm_transmission" params="name">
+    <transmission name="${name}_trans_1">
       <type>transmission_interface/SimpleTransmission</type>
-			<actuator name="${name}_motor_1">
+      <actuator name="${name}_motor_1">
         <hardwareInterface>EffortJointInterface</hardwareInterface>
         <mechanicalReduction>1</mechanicalReduction>
       </actuator>
-			<joint name="${name}_joint_1"/>
-		</transmission>
-		<transmission name="${name}_trans_2">
+      <joint name="${name}_joint_1"/>
+    </transmission>
+    <transmission name="${name}_trans_2">
       <type>transmission_interface/SimpleTransmission</type>
-			<actuator name="${name}_motor_2">
+      <actuator name="${name}_motor_2">
         <hardwareInterface>EffortJointInterface</hardwareInterface>
         <mechanicalReduction>1</mechanicalReduction>
       </actuator>
-			<joint name="${name}_joint_2"/>
-		</transmission>
-		<transmission name="${name}_trans_3">
+      <joint name="${name}_joint_2"/>
+    </transmission>
+    <transmission name="${name}_trans_3">
       <type>transmission_interface/SimpleTransmission</type>
-			<actuator name="${name}_motor_3">
+      <actuator name="${name}_motor_3">
         <hardwareInterface>EffortJointInterface</hardwareInterface>
         <mechanicalReduction>1</mechanicalReduction>
       </actuator>
-			<joint name="${name}_joint_3"/>
-		</transmission>
-		<transmission name="${name}_trans_4">
+      <joint name="${name}_joint_3"/>
+    </transmission>
+    <transmission name="${name}_trans_4">
       <type>transmission_interface/SimpleTransmission</type>
-			<actuator name="${name}_motor_4">
+      <actuator name="${name}_motor_4">
         <hardwareInterface>EffortJointInterface</hardwareInterface>
         <mechanicalReduction>1</mechanicalReduction>
       </actuator>
-			<joint name="${name}_joint_4"/>
-		</transmission>
-		<transmission name="${name}_trans_5">
+      <joint name="${name}_joint_4"/>
+    </transmission>
+    <transmission name="${name}_trans_5">
       <type>transmission_interface/SimpleTransmission</type>
-			<actuator name="${name}_motor_5">
+      <actuator name="${name}_motor_5">
         <hardwareInterface>EffortJointInterface</hardwareInterface>
         <mechanicalReduction>1</mechanicalReduction>
       </actuator>
-			<joint name="${name}_joint_5"/>
-		</transmission>
-	</xacro:macro>
+      <joint name="${name}_joint_5"/>
+    </transmission>
+  </xacro:macro>
 </robot>

File: urdf/youbot_base/base.transmission.xacro (robot description, xacro)
@@ -4,20 +4,20 @@
        xmlns:interface="http://playerstage.sourceforge.net/gazebo/xmlschema/#interface"
        xmlns:xacro="http://ros.org/wiki/xacro">
-	<property name="wheel_mechanical_reduction" value="${624/35 * 80/18}" />
-	<property name="caster_mechanical_reduction" value="${624/35 * 80/18}" />
+  <property name="wheel_mechanical_reduction" value="${624/35 * 80/18}" />
+  <property name="caster_mechanical_reduction" value="${624/35 * 80/18}" />
   <property name="" value="0.360" />
-	<xacro:macro name="youbot_base_transmission">
-	<!-- front left wheel -->
-		<transmission name="wheel_trans_fl">
+  <xacro:macro name="youbot_base_transmission">
+  <!-- front left wheel -->
+    <transmission name="wheel_trans_fl">
       <type>transmission_interface/SimpleTransmission</type>
-			<actuator name="wheel_motor_fl">
+      <actuator name="wheel_motor_fl">
         <hardwareInterface>VelocityJointInterface</hardwareInterface>
         <mechanicalReduction>${wheel_mechanical_reduction}</mechanicalReduction>
       </actuator>
-			<joint name="wheel_joint_fl" />
-		</transmission>
-		<transmission name="caster_trans_fl">
+      <joint name="wheel_joint_fl" />
+    </transmission>
+    <transmission name="caster_trans_fl">
       <type>transmission_interface/SimpleTransmission</type>
-   	  <actuator name="caster_motor_fl">
+       <actuator name="caster_motor_fl">
         <hardwareInterface>VelocityJointInterface</hardwareInterface>
         <mechanicalReduction>${caster_mechanical_reduction}</mechanicalReduction>
@@ -25,14 +25,14 @@
       <joint name="caster_joint_fl" />
     </transmission>
-	  <!-- front right wheel -->
-	  <transmission name="wheel_trans_fr">
+    <!-- front right wheel -->
+    <transmission name="wheel_trans_fr">
       <type>transmission_interface/SimpleTransmission</type>
-		  <actuator name="wheel_motor_fr">
+      <actuator name="wheel_motor_fr">
         <hardwareInterface>VelocityJointInterface</hardwareInterface>
         <mechanicalReduction>${wheel_mechanical_reduction}</mechanicalReduction>
       </actuator>
-		  <joint name="wheel_joint_fr" />
-	  </transmission>
-	  <transmission name="caster_trans_fr">
+      <joint name="wheel_joint_fr" />
+    </transmission>
+    <transmission name="caster_trans_fr">
       <type>transmission_interface/SimpleTransmission</type>
       <actuator name="caster_motor_fr" >
@@ -40,16 +40,16 @@
         <mechanicalReduction>${caster_mechanical_reduction}</mechanicalReduction>
       </actuator>
-    	<joint name="caster_joint_fr" />
+      <joint name="caster_joint_fr" />
     </transmission>
-	  <!-- back left wheel -->
-	  <transmission name="wheel_trans_bl">
+    <!-- back left wheel -->
+    <transmission name="wheel_trans_bl">
       <type>transmission_interface/SimpleTransmission</type>
-	    <actuator name="wheel_motor_bl" >
+      <actuator name="wheel_motor_bl" >
         <hardwareInterface>VelocityJointInterface</hardwareInterface>
         <mechanicalReduction>${wheel_mechanical_reduction}</mechanicalReduction>
       </actuator>
-	    <joint name="wheel_joint_bl" />
-	  </transmission>
-	  <transmission name="caster_trans_bl">
+      <joint name="wheel_joint_bl" />
+    </transmission>
+    <transmission name="caster_trans_bl">
       <type>transmission_interface/SimpleTransmission</type>
       <actuator name="caster_motor_bl" >
@@ -57,16 +57,16 @@
         <mechanicalReduction>${caster_mechanical_reduction}</mechanicalReduction>
       </actuator>
-    	<joint name="caster_joint_bl" />
+      <joint name="caster_joint_bl" />
     </transmission>
-	  <!-- back right wheel -->
-	  <transmission name="wheel_trans_br">
+    <!-- back right wheel -->
+    <transmission name="wheel_trans_br">
       <type>transmission_interface/SimpleTransmission</type>
-	    <actuator name="wheel_motor_br" >
+      <actuator name="wheel_motor_br" >
         <hardwareInterface>VelocityJointInterface</hardwareInterface>
         <mechanicalReduction>${wheel_mechanical_reduction}</mechanicalReduction>
       </actuator>
-		  <joint name="wheel_joint_br" />
-	  </transmission>
-	  <transmission name="caster_trans_br">
+      <joint name="wheel_joint_br" />
+    </transmission>
+    <transmission name="caster_trans_br">
       <type>transmission_interface/SimpleTransmission</type>
       <actuator name="caster_motor_br" >
@@ -74,5 +74,5 @@
         <mechanicalReduction>${caster_mechanical_reduction}</mechanicalReduction>
       </actuator>
-    	<joint name="caster_joint_br" />
+      <joint name="caster_joint_br" />
     </transmission>
   </xacro:macro>

File: urdf/youbot_gripper/gripper.transmission.xacro (robot description, xacro)
@@ -4,21 +4,21 @@
        xmlns:interface="http://playerstage.sourceforge.net/gazebo/xmlschema/#interface"
        xmlns:xacro="http://ros.org/wiki/xacro">
-	<xacro:macro name="youbot_gripper_transmission" params="name">
-		<transmission name="${name}_finger_l_trans">
+  <xacro:macro name="youbot_gripper_transmission" params="name">
+    <transmission name="${name}_finger_l_trans">
       <type>transmission_interface/SimpleTransmission</type>
-			<actuator name="${name}_finger_l_motor">
+      <actuator name="${name}_finger_l_motor">
         <hardwareInterface>EffortJointInterface</hardwareInterface>
         <mechanicalReduction>1</mechanicalReduction>
       </actuator>
-			<joint name="${name}_finger_joint_l"/>
-		</transmission>
-		<transmission name="${name}_finger_r_trans">
+      <joint name="${name}_finger_joint_l"/>
+    </transmission>
+    <transmission name="${name}_finger_r_trans">
       <type>transmission_interface/SimpleTransmission</type>
-			<actuator name="${name}_finger_r_motor">
+      <actuator name="${name}_finger_r_motor">
         <hardwareInterface>EffortJointInterface</hardwareInterface>
         <mechanicalReduction>1</mechanicalReduction>
       </actuator>
-			<joint name="${name}_finger_joint_r"/>
-		</transmission>
-	</xacro:macro>
+      <joint name="${name}_finger_joint_r"/>
+    </transmission>
+  </xacro:macro>
 </robot>
