Commit message: add hardware interface tag to joints
This is required for ROS Indigo.

File: urdf/youbot_arm/arm.transmission.xacro (robot description, xacro)
@@ -13,5 +13,7 @@
         <mechanicalReduction>1</mechanicalReduction>
       </actuator>
-      <joint name="${name}_joint_1"/>
+      <joint name="${name}_joint_1">
+        <hardwareInterface>EffortJointInterface</hardwareInterface>
+      </joint>
     </transmission>
     <transmission name="${name}_trans_2">
@@ -21,5 +23,7 @@
         <mechanicalReduction>1</mechanicalReduction>
       </actuator>
-      <joint name="${name}_joint_2"/>
+      <joint name="${name}_joint_2">
+        <hardwareInterface>EffortJointInterface</hardwareInterface>
+      </joint>
     </transmission>
     <transmission name="${name}_trans_3">
@@ -29,5 +33,7 @@
         <mechanicalReduction>1</mechanicalReduction>
       </actuator>
-      <joint name="${name}_joint_3"/>
+      <joint name="${name}_joint_3">
+        <hardwareInterface>EffortJointInterface</hardwareInterface>
+      </joint>
     </transmission>
     <transmission name="${name}_trans_4">
@@ -37,5 +43,7 @@
         <mechanicalReduction>1</mechanicalReduction>
       </actuator>
-      <joint name="${name}_joint_4"/>
+      <joint name="${name}_joint_4">
+        <hardwareInterface>EffortJointInterface</hardwareInterface>
+      </joint>
     </transmission>
     <transmission name="${name}_trans_5">
@@ -45,5 +53,7 @@
         <mechanicalReduction>1</mechanicalReduction>
       </actuator>
-      <joint name="${name}_joint_5"/>
+      <joint name="${name}_joint_5">
+        <hardwareInterface>EffortJointInterface</hardwareInterface>
+      </joint>
     </transmission>
   </xacro:macro>

File: urdf/youbot_base/base.transmission.xacro (robot description, xacro)
@@ -15,5 +15,7 @@
         <mechanicalReduction>${wheel_mechanical_reduction}</mechanicalReduction>
       </actuator>
-      <joint name="wheel_joint_fl" />
+      <joint name="wheel_joint_fl">
+        <hardwareInterface>VelocityJointInterface</hardwareInterface>
+      </joint>
     </transmission>
     <transmission name="caster_trans_fl">
@@ -23,5 +25,7 @@
         <mechanicalReduction>${caster_mechanical_reduction}</mechanicalReduction>
       </actuator>
-      <joint name="caster_joint_fl" />
+      <joint name="caster_joint_fl">
+        <hardwareInterface>VelocityJointInterface</hardwareInterface>
+      </joint>
     </transmission>
     <!-- front right wheel -->
@@ -32,5 +36,7 @@
         <mechanicalReduction>${wheel_mechanical_reduction}</mechanicalReduction>
       </actuator>
-      <joint name="wheel_joint_fr" />
+      <joint name="wheel_joint_fr">
+        <hardwareInterface>VelocityJointInterface</hardwareInterface>
+      </joint>
     </transmission>
     <transmission name="caster_trans_fr">
@@ -40,5 +46,7 @@
         <mechanicalReduction>${caster_mechanical_reduction}</mechanicalReduction>
       </actuator>
-      <joint name="caster_joint_fr" />
+      <joint name="caster_joint_fr">
+        <hardwareInterface>VelocityJointInterface</hardwareInterface>
+      </joint>
     </transmission>
     <!-- back left wheel -->
@@ -49,5 +57,7 @@
         <mechanicalReduction>${wheel_mechanical_reduction}</mechanicalReduction>
       </actuator>
-      <joint name="wheel_joint_bl" />
+      <joint name="wheel_joint_bl">
+        <hardwareInterface>VelocityJointInterface</hardwareInterface>
+      </joint>
     </transmission>
     <transmission name="caster_trans_bl">
@@ -57,5 +67,7 @@
         <mechanicalReduction>${caster_mechanical_reduction}</mechanicalReduction>
       </actuator>
-      <joint name="caster_joint_bl" />
+      <joint name="caster_joint_bl">
+        <hardwareInterface>VelocityJointInterface</hardwareInterface>
+      </joint>
     </transmission>
     <!-- back right wheel -->
@@ -66,5 +78,7 @@
         <mechanicalReduction>${wheel_mechanical_reduction}</mechanicalReduction>
       </actuator>
-      <joint name="wheel_joint_br" />
+      <joint name="wheel_joint_br">
+        <hardwareInterface>VelocityJointInterface</hardwareInterface>
+      </joint>
     </transmission>
     <transmission name="caster_trans_br">
@@ -74,5 +88,7 @@
         <mechanicalReduction>${caster_mechanical_reduction}</mechanicalReduction>
       </actuator>
-      <joint name="caster_joint_br" />
+      <joint name="caster_joint_br">
+        <hardwareInterface>VelocityJointInterface</hardwareInterface>
+      </joint>
     </transmission>
   </xacro:macro>

File: urdf/youbot_gripper/gripper.transmission.xacro (robot description, xacro)
@@ -11,5 +11,7 @@
         <mechanicalReduction>1</mechanicalReduction>
       </actuator>
-      <joint name="${name}_finger_joint_l"/>
+      <joint name="${name}_finger_joint_l">
+        <hardwareInterface>EffortJointInterface</hardwareInterface>
+      </joint>
     </transmission>
     <transmission name="${name}_finger_r_trans">
@@ -19,5 +21,7 @@
         <mechanicalReduction>1</mechanicalReduction>
       </actuator>
-      <joint name="${name}_finger_joint_r"/>
+      <joint name="${name}_finger_joint_r">
+        <hardwareInterface>EffortJointInterface</hardwareInterface>
+      </joint>
     </transmission>
   </xacro:macro>
