Commit message: update ASUS Xtion gazebo file for hydro

File: urdf/sensors/asus_xtion_camera.gazebo.xacro (robot description, xacro)
@@ -5,60 +5,39 @@
       xmlns:xacro="http://ros.org/wiki/xacro">
 <xacro:macro name="asus_xtion_camera_gazebo" params="name">
-  <xacro:asus_xtion_depth_camera_gazebo name="${name}" />
-  <xacro:asus_xtion_rgb_camera_gazebo name="${name}" />
-</xacro:macro>
-<xacro:macro name="asus_xtion_depth_camera_gazebo" params="name">
-  <gazebo reference="${name}_depth_frame">
-    <sensor:camera name="${name}_depth_frame_sensor">
-      <imageFormat>R8G8B8</imageFormat>
-      <imageSize>640 480</imageSize>
-      <hfov>57</hfov>
-      <nearClip>0.01</nearClip>
-      <farClip>5</farClip>
-      <updateRate>20.0</updateRate>
+  <gazebo reference="${name}_camera">
+  <sensor type="depth" name="${name}_frame_sensor">
+    <always_on>true</always_on>
+    <update_rate>20.0</update_rate>
+    <camera>
+      <horizontal_fov>${62.0*M_PI/180.0}</horizontal_fov>
+      <image>
+        <format>R8G8B8</format>
+        <width>640</width>
+        <height>480</height>
+      </image>
+      <clip>
+        <near>0.1</near>
+        <far>100</far>
+      </clip>
+    </camera>
+    <plugin name="${name}_depth_frame_controller" filename="libgazebo_ros_openni_kinect.so">
       <baseline>0.2</baseline>
-      <controller:gazebo_ros_camera name="${name}_depth_frame_controller" plugin="libgazebo_ros_camera.so">
-        <alwaysOn>true</alwaysOn>
-        <updateRate>20.0</updateRate>
-        <imageTopicName>/camera/ir/image_raw</imageTopicName>
-        <cameraInfoTopicName>/camera/ir/camera_info</cameraInfoTopicName>
-        <depthImageTopicName>/camera/depth/image_raw</depthImageTopicName>
-        <depthImageInfoTopicName>/camera/depth/camera_info</depthImageInfoTopicName>
-        <pointCloudTopicName>/camera/depth/points</pointCloudTopicName>
-        <frameName>/${name}_depth_optical_frame</frameName>
-        <pointCloudCutoff>0.5</pointCloudCutoff>
-        <distortion_k1>0.00000001</distortion_k1>
-        <distortion_k2>0.00000001</distortion_k2>
-        <distortion_k3>0.00000001</distortion_k3>
-        <distortion_t1>0.00000001</distortion_t1>
-        <distortion_t2>0.00000001</distortion_t2>
-      </controller:gazebo_ros_camera>
-    </sensor:camera>
-  </gazebo>
-</xacro:macro>
-<xacro:macro name="asus_xtion_rgb_camera_gazebo" params="name">
-  <gazebo reference="${name}_rgb_frame">
-    <sensor:camera name="${name}_rgb_frame_sensor">
-      <imageFormat>R8G8B8</imageFormat>
-      <imageSize>640 480</imageSize>
-      <hfov>57</hfov>
-      <nearClip>0.01</nearClip>
-      <farClip>5</farClip>
-      <updateRate>20.0</updateRate>
-      <baseline>0.2</baseline>
-      <controller:gazebo_ros_camera name="${name}_rgb_frame_controller" plugin="libgazebo_ros_camera.so">
-        <alwaysOn>true</alwaysOn>
-        <updateRate>20.0</updateRate>
-        <imageTopicName>/camera/rgb/image_raw</imageTopicName>
-        <cameraInfoTopicName>/camera/rgb/camera_info</cameraInfoTopicName>
-        <frameName>/${name}_rgb_optical_frame</frameName>
-        <pointCloudCutoff>0.5</pointCloudCutoff>
-        <distortion_k1>0.00000001</distortion_k1>
-        <distortion_k2>0.00000001</distortion_k2>
-        <distortion_k3>0.00000001</distortion_k3>
-        <distortion_t1>0.00000001</distortion_t1>
-        <distortion_t2>0.00000001</distortion_t2>
-      </controller:gazebo_ros_camera>
-    </sensor:camera>
+      <alwaysOn>true</alwaysOn>
+      <updateRate>2.0</updateRate>
+      <cameraName>${name}</cameraName>
+      <imageTopicName>/${name}/ir/image_raw</imageTopicName>
+      <cameraInfoTopicName>/${name}/ir/camera_info</cameraInfoTopicName>
+      <depthImageTopicName>/${name}/depth/image_raw</depthImageTopicName>
+      <depthImageInfoTopicName>/${name}/depth/camera_info</depthImageInfoTopicName>
+      <pointCloudTopicName>/${name}/depth/points</pointCloudTopicName>
+      <frameName>${name}_depth_optical_frame</frameName>
+      <pointCloudCutoff>0.5</pointCloudCutoff>
+      <distortionK1>0.00000001</distortionK1>
+      <distortionK2>0.00000001</distortionK2>
+      <distortionK3>0.00000001</distortionK3>
+      <distortionT1>0.00000001</distortionT1>
+      <distortionT2>0.00000001</distortionT2>
+    </plugin>
+  </sensor>
   </gazebo>
 </xacro:macro>
