Commit message: remove material tag (not supported for dae) and correct identation

File: urdf/sensors/hokuyo_urg04_laser.urdf.xacro (robot description, xacro)
@@ -19,16 +19,15 @@
       </inertial>
       <visual>
-      	<origin xyz="0 0 0" rpy="0 0 0" />
-	<geometry>
-		<mesh filename="package://youbot_description/meshes/sensors/hokuyo.dae" />
-	</geometry>
-	<material name="DarkGrey" />
+        <origin xyz="0 0 0" rpy="0 0 0" />
+        <geometry>
+          <mesh filename="package://youbot_description/meshes/sensors/hokuyo.dae" />
+        </geometry>
       </visual>
       <collision>
-		<origin xyz="0 0 0" rpy="0 0 0" />
-		<geometry>
-			<mesh filename="package://youbot_description/meshes/sensors/hokuyo_convex.dae" />
-		</geometry>
-	</collision>
+        <origin xyz="0 0 0" rpy="0 0 0" />
+        <geometry>
+          <mesh filename="package://youbot_description/meshes/sensors/hokuyo_convex.dae" />
+        </geometry>
+      </collision>
     </link>
     <!-- gazebo extensions -->

Commit message: [urdf][sensor] Removed type attr in link

File: urdf/sensors/hokuyo_urg04_laser.urdf.xacro (robot description, xacro)
@@ -12,5 +12,5 @@
       <child link="${name}_link"/>
     </joint>
-    <link name="${name}_link" type="laser">
+    <link name="${name}_link">
       <inertial>
         <mass value="0.16" />
