Commit message: fixed origin of collision mesh
This is for issue mas-group/mas_industrial_robotics#39

File: urdf/misc/arm_pov_mount.urdf.xacro (robot description, xacro)
@@ -19,5 +19,5 @@
       </visual>
       <collision>
-        <origin xyz="0 0 0" rpy="0 0 0" />
+        <origin xyz="-0.015 0.04 -0.055" rpy="0 0 -1.57079633" />
         <geometry>
 			<mesh filename="package://youbot_description/meshes/sensors/arm_pov_mount.dae" scale="0.0001 0.0001 0.0001"/>
