Commit message: add entries from old updated_materials.urdf.xacro

File: urdf/materials.urdf.xacro (robot description, xacro)
@@ -22,3 +22,9 @@
     <color rgba="0.0 1.0 0.0 1.0"/>
   </material>
+  <material name="Blue">
+    <color rgba="0.0 0.0 0.8 1.0"/>
+  </material>
+  <material name="LightGrey">
+    <color rgba="0.82 0.82 0.82 1.0"/>
+  </material>
 </robot>

Commit message: get rid of color warnings in simulation

File: urdf/materials.urdf.xacro (robot description, xacro)
@@ -1,29 +1,29 @@
 <?xml version="1.0"?>
 <robot>
-  <material name="Orange">
+  <material name="youBot/Orange">
     <color rgba="1.0 0.4 0.0 1.0"/>
   </material>
-  <material name="Grey">
+  <material name="youBot/Grey">
     <color rgba="0.7 0.7 0.7 1.0"/>
   </material>
-  <material name="DarkGrey">
+  <material name="youBot/DarkGrey">
     <color rgba="0.3 0.3 0.3 1.0"/>
   </material>
-  <material name="White">
+  <material name="youBot/White">
     <color rgba="1.0 1.0 1.0 1.0"/>
   </material>
-  <material name="Black">
+  <material name="youBot/Black">
     <color rgba="0.0 0.0 0.0 1.0"/>
   </material>
-  <material name="Red">
+  <material name="youBot/Red">
     <color rgba="1.0 0.0 0.0 1.0"/>
   </material>
-  <material name="Green">
+  <material name="youBot/Green">
     <color rgba="0.0 1.0 0.0 1.0"/>
   </material>
-  <material name="Blue">
+  <material name="youBot/Blue">
     <color rgba="0.0 0.0 0.8 1.0"/>
   </material>
-  <material name="LightGrey">
+  <material name="youBot/LightGrey">
     <color rgba="0.82 0.82 0.82 1.0"/>
   </material>

File: urdf/misc/camera_tower.urdf.xacro (robot description, xacro)
@@ -19,5 +19,5 @@
           <box size="${camera_tower_depth} ${camera_tower_width} ${camera_tower_height}"/>
         </geometry>
-        <material name="LightGrey" />
+        <material name="youBot/LightGrey" />
       </visual>
       <collision>

File: urdf/youbot_arm/arm.gazebo.xacro (robot description, xacro)
@@ -6,25 +6,19 @@
 	<xacro:macro name="youbot_arm_gazebo" params="name">
 		<gazebo reference="${name}_link_0">
-			<material value="youbot/DarkGrey" />
 			<turnGravityOff>false</turnGravityOff>
 		</gazebo>
 		<gazebo reference="${name}_link_1">
-			<!--<material value="youbot/Orange" />-->
 			<turnGravityOff>false</turnGravityOff>
 		</gazebo>
 		<gazebo reference="${name}_link_2">
-			<!--<material value="youbot/Orange" />-->
 			<turnGravityOff>false</turnGravityOff>
 		</gazebo>
 		<gazebo reference="${name}_link_3">
-			<!--<material value="youbot/Orange" />-->
 			<turnGravityOff>false</turnGravityOff>
 		</gazebo>
 		<gazebo reference="${name}_link_4">
-			<!--<material value="youbot/Orange" />-->
 			<turnGravityOff>false</turnGravityOff>
 		</gazebo>
 		<gazebo reference="${name}_link_5">
-			<!--<material value="youbot/DarkGrey" />-->
 			<turnGravityOff>false</turnGravityOff>
 		</gazebo>

File: urdf/youbot_arm/arm.urdf.xacro (robot description, xacro)
@@ -26,5 +26,5 @@
 					<mesh filename="package://youbot_description/meshes/youbot_arm/arm0.dae" />
 				</geometry>
-				<material name="DarkGrey" />
+				<material name="youBot/DarkGrey" />
 			</visual>
 			<collision>
@@ -65,5 +65,5 @@
 					<mesh filename="package://youbot_description/meshes/youbot_arm/arm1.dae" />
 				</geometry>
-				<!--<material name="Orange" />-->
+				<material name="youBot/Orange" />
 			</visual>
 			<collision>
@@ -97,5 +97,4 @@
 					<mesh filename="package://youbot_description/meshes/youbot_arm/arm2.dae" />
 				</geometry>
-				<material name="Orange" />
 			</visual>
 			<collision>
@@ -137,5 +136,5 @@
 					<mesh filename="package://youbot_description/meshes/youbot_arm/arm3.dae" />
 				</geometry>
-				<material name="Orange" />
+				<material name="youBot/Orange" />
 			</visual>
 			<collision>
@@ -169,5 +168,5 @@
 					<mesh filename="package://youbot_description/meshes/youbot_arm/arm4.dae" />
 				</geometry>
-				<material name="Orange" />
+				<material name="youBot/Orange" />
 			</visual>
 			<collision>
@@ -201,5 +200,5 @@
 					<mesh filename="package://youbot_description/meshes/youbot_arm/arm5.dae" />
 				</geometry>
-				<material name="DarkGrey" />
+				<material name="youBot/DarkGrey" />
 			</visual>
 			<collision>

File: urdf/youbot_base/base.gazebo.xacro (robot description, xacro)
@@ -6,41 +6,32 @@
   <xacro:macro name="youbot_base_gazebo">
     <gazebo reference="youbot_base">
-      <material value="youbot/DarkGrey" />
     </gazebo>
     <!-- front left wheel -->
     <gazebo reference="wheel_link_fl">
-      <material value="youbot/Orange" />
       <kp>1000000</kp>
       <kd>100</kd>
     </gazebo>
     <gazebo reference="caster_link_fl">
-      <material value="youbot/Orange" />
     </gazebo>
     <!-- front right wheel -->
     <gazebo reference="wheel_link_fr">
-      <material value="youbot/Orange" />
       <kp>1000000</kp>
       <kd>100</kd>
     </gazebo>
     <gazebo reference="caster_link_fr">
-      <material value="youbot/Orange" />
     </gazebo>
     <!-- back left wheel -->
     <gazebo reference="wheel_link_bl">
-      <material value="youbot/Orange" />
       <kp>1000000</kp>
       <kd>100</kd>
     </gazebo>
     <gazebo reference="caster_link_bl">
-      <material value="youbot/Orange" />
     </gazebo>
     <!-- back right wheel -->
     <gazebo reference="wheel_link_br">
-      <material value="youbot/Orange" />
       <kp>1000000</kp>
       <kd>100</kd>
     </gazebo>
     <gazebo reference="caster_link_br">
-      <material value="youbot/Orange" />
     </gazebo>
     <!-- position controller -->

File: urdf/youbot_base/base.urdf.xacro (robot description, xacro)
@@ -4,5 +4,4 @@
        xmlns:interface="http://playerstage.sourceforge.net/gazebo/xmlschema/#interface"
        xmlns:xacro="http://ros.org/wiki/xacro">
-  <!-- sensors -->
   <xacro:include filename="$(find youbot_description)/urdf/youbot_base/base.gazebo.xacro"/>
   <xacro:include filename="$(find youbot_description)/urdf/youbot_base/base.transmission.xacro"/>
@@ -44,5 +43,5 @@
           <box size="0.001 0.001 0.001"/>
         </geometry>
-        <material name="Red"/>
+        <material name="youBot/Red"/>
       </visual>
       <collision>
@@ -69,5 +68,5 @@
           <mesh filename="package://youbot_description/meshes/youbot_base/base.dae"/>
         </geometry>
-        <material name="DarkGrey"/>
+        <material name="youBot/DarkGrey"/>
       </visual>
       <collision>
@@ -117,5 +116,5 @@
           <sphere radius="${wheel_radius}"/>
         </geometry>
-        <material name="Orange"/>
+        <material name="youBot/Orange"/>
       </visual>
       <collision>
@@ -164,5 +163,5 @@
           <sphere radius="${wheel_radius}"/>
         </geometry>
-        <material name="Orange"/>
+        <material name="youBot/Orange"/>
       </visual>
       <collision>
@@ -212,5 +211,5 @@
           <sphere radius="${wheel_radius}"/>
         </geometry>
-        <material name="Orange"/>
+        <material name="youBot/Orange"/>
       </visual>
       <collision>
@@ -259,5 +258,5 @@
           <sphere radius="${wheel_radius}"/>
         </geometry>
-        <material name="Orange"/>
+        <material name="youBot/Orange"/>
       </visual>
       <collision>
