Commit message: set correct mass of the plate
source: http://www.youbot-store.com/developers/documentation/kuka-youbot-kinematics-dynamics-and-3d-model

File: urdf/youbot_plate/plate.urdf.xacro (robot description, xacro)
@@ -14,5 +14,5 @@
 			<inertial>
 				<origin xyz="0 0 0" rpy="0 0 0"/>
-				<mass value="1"/>
+				<mass value="2.397"/>
 				<inertia ixx="0.01" ixy="0" ixz="0" iyy="0.01" iyz="0" izz="0.01" />
 			</inertial>
