Commit message: updated xacro files for the current version of ros kinetic

File: controller/ros_controller.urdf.xacro (robot description, xacro)
@@ -4,5 +4,7 @@
        xmlns:interface="http://playerstage.sourceforge.net/gazebo/xmlschema/#interface">
   <gazebo>
-    <plugin name="gazebo_ros_controller" filename="libgazebo_ros_control.so" />
+    <plugin name="gazebo_ros_controller" filename="libgazebo_ros_control.so">
+    <legacyModeNS>true</legacyModeNS>
+    </plugin>
   </gazebo>
 </robot>

File: urdf/youbot_base/base.urdf.xacro (robot description, xacro)
@@ -33,9 +33,10 @@
   <xacro:macro name="youbot_base" params="name">
     <link name="${name}_footprint">
-      <inertial>
+      <!--<inertial>
         <mass value="0.1"/>
         <origin xyz="0 0 ${-base_size_z / 2.0}" rpy="0 0 0"/>
         <inertia ixx="1.0" ixy="0.0" ixz="0.0" iyy="1.0" iyz="0.0" izz="1.0"/>
       </inertial>
+    -->
       <visual>
         <origin xyz="0 0 0" rpy="0 0 0"/>
